Commit message: update description

File: src/omni_1_description/urdf/omni_1.urdf (robot description, URDF)
Before this commit: robot urdf, 4 links, 3 joints
Links:
- removed link base_linkv2_1
- removed link wheel-framev2_1
- removed link wheel-framev2_2
- removed link wheel-framev2_3
- added link base_link, mass 4.810857321318848; collision mesh filename=package://omni_1_description/meshes/base_link.stl scale=0.001 0.001 0.001; visual mesh filename=package://omni_1_description/meshes/base_link.stl scale=0.001 0.001 0.001
- added link wheel-frame0, mass 0.5173431185653956; collision mesh filename=package://omni_1_description/meshes/wheel-frame0.stl scale=0.001 0.001 0.001; visual mesh filename=package://omni_1_description/meshes/wheel-frame0.stl scale=0.001 0.001 0.001
- added link wheel-frame120, mass 0.5173431185653956; collision mesh filename=package://omni_1_description/meshes/wheel-frame120.stl scale=0.001 0.001 0.001; visual mesh filename=package://omni_1_description/meshes/wheel-frame120.stl scale=0.001 0.001 0.001
- added link wheel-frame240, mass 0.5173431185653956; collision mesh filename=package://omni_1_description/meshes/wheel-frame240.stl scale=0.001 0.001 0.001; visual mesh filename=package://omni_1_description/meshes/wheel-frame240.stl scale=0.001 0.001 0.001
Joints:
- joint Revolute11: child wheel-framev2_2 -> wheel-frame120; parent base_linkv2_1 -> base_link
- joint Revolute12: child wheel-framev2_3 -> wheel-frame240; parent base_linkv2_1 -> base_link
- joint Revolute8: child wheel-framev2_1 -> wheel-frame0; parent base_linkv2_1 -> base_link

Commit message: update urdf, wheel frames fixed

File: src/omni_1_description/urdf/omni_1.urdf (robot description, URDF)
Before this commit: robot urdf, 4 links, 3 joints
Links:
- link base_link: mass 4.810857321318848 -> 4.8
- link wheel-frame0: mass 0.5173431185653956 -> 0.5
- link wheel-frame120: mass 0.5173431185653956 -> 0.5
- link wheel-frame240: mass 0.5173431185653956 -> 0.5
Joints:
- removed joint Revolute11
- removed joint Revolute12
- removed joint Revolute8
- added joint wheel-frame0: type revolute, parent base_link, child wheel-frame0, origin xyz=0.0 -0.1 0.0 rpy=0 0 0, axis 0.0 -1.0 0.0, limit lower=-3.14159 upper=3.14159 effort=100 velocity=100
- added joint wheel-frame120: type revolute, parent base_link, child wheel-frame120, origin xyz=0.08660254038 0.05 0.0 rpy=0 0 2.094395102, axis 0.0 -1.0 0.0, limit lower=-3.14159 upper=3.14159 effort=100 velocity=100
- added joint wheel-frame240: type revolute, parent base_link, child wheel-frame240, origin xyz=-0.08660254038 0.05 0.0 rpy=0 0 4.188790205, axis 0.0 -1.0 0.0, limit lower=-3.14159 upper=3.14159 effort=100 velocity=100

Commit message: added 1 roller, not fully

File: src/omni_1_description/urdf/omni_1.urdf (robot description, URDF)
Before this commit: robot urdf, 4 links, 3 joints
Links:
- added link roller-0-0, mass 0.02; collision mesh filename=package://omni_1_description/meshes/roller.stl scale=0.001 0.001 0.001; visual mesh filename=package://omni_1_description/meshes/roller.stl scale=0.001 0.001 0.001
Joints:
- added joint wheel0-roller0: type continuous, parent wheel-frame0, child roller-0-0, origin xyz=0.0 0.013 0.03 rpy=0 0 0, axis 1.0 0.0 0.0
- joint wheel-frame0: limit lower=-3.14159 upper=3.14159 effort=100 velocity=100 -> effort=100 velocity=100; type revolute -> continuous
- joint wheel-frame120: limit lower=-3.14159 upper=3.14159 effort=100 velocity=100 -> effort=100 velocity=100; type revolute -> continuous
- joint wheel-frame240: limit lower=-3.14159 upper=3.14159 effort=100 velocity=100 -> effort=100 velocity=100; type revolute -> continuous

Commit message: 1 ceo tocak

File: src/omni_1_description/urdf/omni_1.urdf (robot description, URDF)
Before this commit: robot urdf, 5 links, 4 joints
Links:
- added link roller-0-1, mass 0.02; collision mesh filename=package://omni_1_description/meshes/roller.stl scale=0.001 0.001 0.001; visual mesh filename=package://omni_1_description/meshes/roller.stl scale=0.001 0.001 0.001
- added link roller-0-2, mass 0.02; collision mesh filename=package://omni_1_description/meshes/roller.stl scale=0.001 0.001 0.001; visual mesh filename=package://omni_1_description/meshes/roller.stl scale=0.001 0.001 0.001
- added link roller-0-3, mass 0.02; collision mesh filename=package://omni_1_description/meshes/roller.stl scale=0.001 0.001 0.001; visual mesh filename=package://omni_1_description/meshes/roller.stl scale=0.001 0.001 0.001
- added link roller-0-4, mass 0.02; collision mesh filename=package://omni_1_description/meshes/roller.stl scale=0.001 0.001 0.001; visual mesh filename=package://omni_1_description/meshes/roller.stl scale=0.001 0.001 0.001
- added link roller-0-5, mass 0.02; collision mesh filename=package://omni_1_description/meshes/roller.stl scale=0.001 0.001 0.001; visual mesh filename=package://omni_1_description/meshes/roller.stl scale=0.001 0.001 0.001
Joints:
- added joint wheel0-roller1: type continuous, parent wheel-frame0, child roller-0-1, origin xyz=0.0207846 0.013 -0.012 rpy=0 2.094395102 0, axis 1.0 0.0 0.0
- added joint wheel0-roller2: type continuous, parent wheel-frame0, child roller-0-2, origin xyz=-0.0207846 0.013 -0.012 rpy=0 4.188790205 0, axis 1.0 0.0 0.0
- added joint wheel0-roller3: type continuous, parent wheel-frame0, child roller-0-3, origin xyz=0.0207846 -0.013 0.012 rpy=0 1.0471975512 0, axis 1.0 0.0 0.0
- added joint wheel0-roller4: type continuous, parent wheel-frame0, child roller-0-4, origin xyz=0.0 -0.013 -0.024 rpy=0 3.1415926536 0, axis 1.0 0.0 0.0
- added joint wheel0-roller5: type continuous, parent wheel-frame0, child roller-0-5, origin xyz=-0.0207846 -0.013 0.012 rpy=0 5.235987756 0, axis 1.0 0.0 0.0
- joint wheel0-roller0: origin xyz=0.0 0.013 0.03 rpy=0 0 0 -> xyz=0.0 0.013 0.024 rpy=0 0 0

Commit message: omniwheels urdf working

File: src/omni_1_description/urdf/omni_1.urdf (robot description, URDF)
Before this commit: robot urdf, 10 links, 9 joints
Links:
- added link roller-1-0, mass 0.02; collision mesh filename=package://omni_1_description/meshes/roller.stl scale=0.001 0.001 0.001; visual mesh filename=package://omni_1_description/meshes/roller.stl scale=0.001 0.001 0.001
- added link roller-1-1, mass 0.02; collision mesh filename=package://omni_1_description/meshes/roller.stl scale=0.001 0.001 0.001; visual mesh filename=package://omni_1_description/meshes/roller.stl scale=0.001 0.001 0.001
- added link roller-1-2, mass 0.02; collision mesh filename=package://omni_1_description/meshes/roller.stl scale=0.001 0.001 0.001; visual mesh filename=package://omni_1_description/meshes/roller.stl scale=0.001 0.001 0.001
- added link roller-1-3, mass 0.02; collision mesh filename=package://omni_1_description/meshes/roller.stl scale=0.001 0.001 0.001; visual mesh filename=package://omni_1_description/meshes/roller.stl scale=0.001 0.001 0.001
- added link roller-1-4, mass 0.02; collision mesh filename=package://omni_1_description/meshes/roller.stl scale=0.001 0.001 0.001; visual mesh filename=package://omni_1_description/meshes/roller.stl scale=0.001 0.001 0.001
- added link roller-1-5, mass 0.02; collision mesh filename=package://omni_1_description/meshes/roller.stl scale=0.001 0.001 0.001; visual mesh filename=package://omni_1_description/meshes/roller.stl scale=0.001 0.001 0.001
- added link roller-2-0, mass 0.02; collision mesh filename=package://omni_1_description/meshes/roller.stl scale=0.001 0.001 0.001; visual mesh filename=package://omni_1_description/meshes/roller.stl scale=0.001 0.001 0.001
- added link roller-2-1, mass 0.02; collision mesh filename=package://omni_1_description/meshes/roller.stl scale=0.001 0.001 0.001; visual mesh filename=package://omni_1_description/meshes/roller.stl scale=0.001 0.001 0.001
- added link roller-2-2, mass 0.02; collision mesh filename=package://omni_1_description/meshes/roller.stl scale=0.001 0.001 0.001; visual mesh filename=package://omni_1_description/meshes/roller.stl scale=0.001 0.001 0.001
- added link roller-2-3, mass 0.02; collision mesh filename=package://omni_1_description/meshes/roller.stl scale=0.001 0.001 0.001; visual mesh filename=package://omni_1_description/meshes/roller.stl scale=0.001 0.001 0.001
- added link roller-2-4, mass 0.02; collision mesh filename=package://omni_1_description/meshes/roller.stl scale=0.001 0.001 0.001; visual mesh filename=package://omni_1_description/meshes/roller.stl scale=0.001 0.001 0.001
- added link roller-2-5, mass 0.02; collision mesh filename=package://omni_1_description/meshes/roller.stl scale=0.001 0.001 0.001; visual mesh filename=package://omni_1_description/meshes/roller.stl scale=0.001 0.001 0.001
Joints:
- added joint wheel120-roller0: type continuous, parent wheel-frame120, child roller-1-0, origin xyz=0.0 0.013 0.024 rpy=0 0 0, axis 1.0 0.0 0.0
- added joint wheel120-roller1: type continuous, parent wheel-frame120, child roller-1-1, origin xyz=0.0207846 0.013 -0.012 rpy=0 2.094395102 0, axis 1.0 0.0 0.0
- added joint wheel120-roller2: type continuous, parent wheel-frame120, child roller-1-2, origin xyz=-0.0207846 0.013 -0.012 rpy=0 4.188790205 0, axis 1.0 0.0 0.0
- added joint wheel120-roller3: type continuous, parent wheel-frame120, child roller-1-3, origin xyz=0.0207846 -0.013 0.012 rpy=0 1.0471975512 0, axis 1.0 0.0 0.0
- added joint wheel120-roller4: type continuous, parent wheel-frame120, child roller-1-4, origin xyz=0.0 -0.013 -0.024 rpy=0 3.1415926536 0, axis 1.0 0.0 0.0
- added joint wheel120-roller5: type continuous, parent wheel-frame120, child roller-1-5, origin xyz=-0.0207846 -0.013 0.012 rpy=0 5.235987756 0, axis 1.0 0.0 0.0
- added joint wheel240-roller0: type continuous, parent wheel-frame240, child roller-2-0, origin xyz=0.0 0.013 0.024 rpy=0 0 0, axis 1.0 0.0 0.0
- added joint wheel240-roller1: type continuous, parent wheel-frame240, child roller-2-1, origin xyz=0.0207846 0.013 -0.012 rpy=0 2.094395102 0, axis 1.0 0.0 0.0
- added joint wheel240-roller2: type continuous, parent wheel-frame240, child roller-2-2, origin xyz=-0.0207846 0.013 -0.012 rpy=0 4.188790205 0, axis 1.0 0.0 0.0
- added joint wheel240-roller3: type continuous, parent wheel-frame240, child roller-2-3, origin xyz=0.0207846 -0.013 0.012 rpy=0 1.0471975512 0, axis 1.0 0.0 0.0
- added joint wheel240-roller4: type continuous, parent wheel-frame240, child roller-2-4, origin xyz=0.0 -0.013 -0.024 rpy=0 3.1415926536 0, axis 1.0 0.0 0.0
- added joint wheel240-roller5: type continuous, parent wheel-frame240, child roller-2-5, origin xyz=-0.0207846 -0.013 0.012 rpy=0 5.235987756 0, axis 1.0 0.0 0.0

Commit message: novi proto u webots, ali mora da se pojednostave stl-ovi dosta

File: src/omni_1_description/urdf/omni_1.urdf (robot description, URDF)
Before this commit: robot urdf, 22 links, 21 joints
Links:
- link base_link: geometry collision mesh filename=package://omni_1_description/meshes/base_link.stl scale=1 1 1; visual mesh filename=package://omni_1_description/meshes/base_link.stl scale=1 1 1
- link roller-0-0: geometry collision mesh filename=package://omni_1_description/meshes/roller.stl scale=1 1 1; visual mesh filename=package://omni_1_description/meshes/roller.stl scale=1 1 1
- link roller-0-1: geometry collision mesh filename=package://omni_1_description/meshes/roller.stl scale=1 1 1; visual mesh filename=package://omni_1_description/meshes/roller.stl scale=1 1 1
- link roller-0-2: geometry collision mesh filename=package://omni_1_description/meshes/roller.stl scale=1 1 1; visual mesh filename=package://omni_1_description/meshes/roller.stl scale=1 1 1
- link roller-0-3: geometry collision mesh filename=package://omni_1_description/meshes/roller.stl scale=1 1 1; visual mesh filename=package://omni_1_description/meshes/roller.stl scale=1 1 1
- link roller-0-4: geometry collision mesh filename=package://omni_1_description/meshes/roller.stl scale=1 1 1; visual mesh filename=package://omni_1_description/meshes/roller.stl scale=1 1 1
- link roller-0-5: geometry collision mesh filename=package://omni_1_description/meshes/roller.stl scale=1 1 1; visual mesh filename=package://omni_1_description/meshes/roller.stl scale=1 1 1
- link roller-1-0: geometry collision mesh filename=package://omni_1_description/meshes/roller.stl scale=1 1 1; visual mesh filename=package://omni_1_description/meshes/roller.stl scale=1 1 1
- link roller-1-1: geometry collision mesh filename=package://omni_1_description/meshes/roller.stl scale=1 1 1; visual mesh filename=package://omni_1_description/meshes/roller.stl scale=1 1 1
- link roller-1-2: geometry collision mesh filename=package://omni_1_description/meshes/roller.stl scale=1 1 1; visual mesh filename=package://omni_1_description/meshes/roller.stl scale=1 1 1
- link roller-1-3: geometry collision mesh filename=package://omni_1_description/meshes/roller.stl scale=1 1 1; visual mesh filename=package://omni_1_description/meshes/roller.stl scale=1 1 1
- link roller-1-4: geometry collision mesh filename=package://omni_1_description/meshes/roller.stl scale=1 1 1; visual mesh filename=package://omni_1_description/meshes/roller.stl scale=1 1 1
- link roller-1-5: geometry collision mesh filename=package://omni_1_description/meshes/roller.stl scale=1 1 1; visual mesh filename=package://omni_1_description/meshes/roller.stl scale=1 1 1
- link roller-2-0: geometry collision mesh filename=package://omni_1_description/meshes/roller.stl scale=1 1 1; visual mesh filename=package://omni_1_description/meshes/roller.stl scale=1 1 1
- link roller-2-1: geometry collision mesh filename=package://omni_1_description/meshes/roller.stl scale=1 1 1; visual mesh filename=package://omni_1_description/meshes/roller.stl scale=1 1 1
- link roller-2-2: geometry collision mesh filename=package://omni_1_description/meshes/roller.stl scale=1 1 1; visual mesh filename=package://omni_1_description/meshes/roller.stl scale=1 1 1
- link roller-2-3: geometry collision mesh filename=package://omni_1_description/meshes/roller.stl scale=1 1 1; visual mesh filename=package://omni_1_description/meshes/roller.stl scale=1 1 1
- link roller-2-4: geometry collision mesh filename=package://omni_1_description/meshes/roller.stl scale=1 1 1; visual mesh filename=package://omni_1_description/meshes/roller.stl scale=1 1 1
- link roller-2-5: geometry collision mesh filename=package://omni_1_description/meshes/roller.stl scale=1 1 1; visual mesh filename=package://omni_1_description/meshes/roller.stl scale=1 1 1
- link wheel-frame0: geometry collision mesh filename=package://omni_1_description/meshes/wheel_frame.stl scale=1 1 1; visual mesh filename=package://omni_1_description/meshes/wheel_frame.stl scale=1 1 1
- link wheel-frame120: geometry collision mesh filename=package://omni_1_description/meshes/wheel_frame.stl scale=1 1 1; visual mesh filename=package://omni_1_description/meshes/wheel_frame.stl scale=1 1 1
- link wheel-frame240: geometry collision mesh filename=package://omni_1_description/meshes/wheel_frame.stl scale=1 1 1; visual mesh filename=package://omni_1_description/meshes/wheel_frame.stl scale=1 1 1

Commit message: nije jos dobar robot, preskacu roleri ponekad

File: src/omni_1_description/urdf/omni_1.urdf (robot description, URDF)
Before this commit: robot omni-1, 22 links, 21 joints
Links:
- removed link wheel-frame0
- removed link wheel-frame120
- removed link wheel-frame240
- added link wheel-frame180, mass 0.1; collision mesh filename=package://omni_1_description/meshes/wheel_frame.stl scale=1 1 1; visual mesh filename=package://omni_1_description/meshes/wheel_frame.stl scale=1 1 1
- added link wheel-frame300, mass 0.1; collision mesh filename=package://omni_1_description/meshes/wheel_frame.stl scale=1 1 1; visual mesh filename=package://omni_1_description/meshes/wheel_frame.stl scale=1 1 1
- added link wheel-frame60, mass 0.1; collision mesh filename=package://omni_1_description/meshes/wheel_frame.stl scale=1 1 1; visual mesh filename=package://omni_1_description/meshes/wheel_frame.stl scale=1 1 1
- link base_link: mass 4.8 -> 0.7
- link roller-0-0: mass 0.02 -> 0.002
- link roller-0-1: mass 0.02 -> 0.002
- link roller-0-2: mass 0.02 -> 0.002
- link roller-0-3: mass 0.02 -> 0.002
- link roller-0-4: mass 0.02 -> 0.002
- link roller-0-5: mass 0.02 -> 0.002
- link roller-1-0: mass 0.02 -> 0.002
- link roller-1-1: mass 0.02 -> 0.002
- link roller-1-2: mass 0.02 -> 0.002
- link roller-1-3: mass 0.02 -> 0.002
- link roller-1-4: mass 0.02 -> 0.002
- link roller-1-5: mass 0.02 -> 0.002
- link roller-2-0: mass 0.02 -> 0.002
- link roller-2-1: mass 0.02 -> 0.002
- link roller-2-2: mass 0.02 -> 0.002
- link roller-2-3: mass 0.02 -> 0.002
- link roller-2-4: mass 0.02 -> 0.002
- link roller-2-5: mass 0.02 -> 0.002
Joints:
- removed joint wheel-frame0
- removed joint wheel-frame120
- removed joint wheel-frame240
- removed joint wheel0-roller0
- removed joint wheel0-roller1
- removed joint wheel0-roller2
- removed joint wheel0-roller3
- removed joint wheel0-roller4
- removed joint wheel0-roller5
- removed joint wheel120-roller0
- removed joint wheel120-roller1
- removed joint wheel120-roller2
- removed joint wheel120-roller3
- removed joint wheel120-roller4
- removed joint wheel120-roller5
- removed joint wheel240-roller0
- removed joint wheel240-roller1
- removed joint wheel240-roller2
- removed joint wheel240-roller3
- removed joint wheel240-roller4
- removed joint wheel240-roller5
- added joint wheel-frame180: type continuous, parent base_link, child wheel-frame180, origin xyz=-0.1 0.0 0.0 rpy=0 0 1.570796327, axis 0.0 -1.0 0.0, limit effort=10 velocity=10
- added joint wheel-frame300: type continuous, parent base_link, child wheel-frame300, origin xyz=0.05 -0.08660254038 0. rpy=0 0 -2.617993878, axis 0.0 -1.0 0.0, limit effort=10 velocity=10
- added joint wheel-frame60: type continuous, parent base_link, child wheel-frame60, origin xyz=0.05 0.08660254038 0.0 rpy=0 0 -0.5235987756, axis 0.0 -1.0 0.0, limit effort=10 velocity=10
- added joint wheel180-roller0: type continuous, parent wheel-frame180, child roller-1-0, origin xyz=0.0 0.013 0.024 rpy=0 0 0, axis 1.0 0.0 0.0
- added joint wheel180-roller1: type continuous, parent wheel-frame180, child roller-1-1, origin xyz=0.0207846 0.013 -0.012 rpy=0 2.094395102 0, axis 1.0 0.0 0.0
- added joint wheel180-roller2: type continuous, parent wheel-frame180, child roller-1-2, origin xyz=-0.0207846 0.013 -0.012 rpy=0 4.188790205 0, axis 1.0 0.0 0.0
- added joint wheel180-roller3: type continuous, parent wheel-frame180, child roller-1-3, origin xyz=0.0207846 -0.013 0.012 rpy=0 1.0471975512 0, axis 1.0 0.0 0.0
- added joint wheel180-roller4: type continuous, parent wheel-frame180, child roller-1-4, origin xyz=0.0 -0.013 -0.024 rpy=0 3.1415926536 0, axis 1.0 0.0 0.0
- added joint wheel180-roller5: type continuous, parent wheel-frame180, child roller-1-5, origin xyz=-0.0207846 -0.013 0.012 rpy=0 5.235987756 0, axis 1.0 0.0 0.0
- added joint wheel300-roller0: type continuous, parent wheel-frame300, child roller-2-0, origin xyz=0.0 0.013 0.024 rpy=0 0 0, axis 1.0 0.0 0.0
- added joint wheel300-roller1: type continuous, parent wheel-frame300, child roller-2-1, origin xyz=0.0207846 0.013 -0.012 rpy=0 2.094395102 0, axis 1.0 0.0 0.0
- added joint wheel300-roller2: type continuous, parent wheel-frame300, child roller-2-2, origin xyz=-0.0207846 0.013 -0.012 rpy=0 4.188790205 0, axis 1.0 0.0 0.0
- added joint wheel300-roller3: type continuous, parent wheel-frame300, child roller-2-3, origin xyz=0.0207846 -0.013 0.012 rpy=0 1.0471975512 0, axis 1.0 0.0 0.0
- added joint wheel300-roller4: type continuous, parent wheel-frame300, child roller-2-4, origin xyz=0.0 -0.013 -0.024 rpy=0 3.1415926536 0, axis 1.0 0.0 0.0
- added joint wheel300-roller5: type continuous, parent wheel-frame300, child roller-2-5, origin xyz=-0.0207846 -0.013 0.012 rpy=0 5.235987756 0, axis 1.0 0.0 0.0
- added joint wheel60-roller0: type continuous, parent wheel-frame60, child roller-0-0, origin xyz=0.0 0.013 0.024 rpy=0 0 0, axis 1.0 0.0 0.0
- added joint wheel60-roller1: type continuous, parent wheel-frame60, child roller-0-1, origin xyz=0.0207846 0.013 -0.012 rpy=0 2.094395102 0, axis 1.0 0.0 0.0
- added joint wheel60-roller2: type continuous, parent wheel-frame60, child roller-0-2, origin xyz=-0.0207846 0.013 -0.012 rpy=0 4.188790205 0, axis 1.0 0.0 0.0
- added joint wheel60-roller3: type continuous, parent wheel-frame60, child roller-0-3, origin xyz=0.0207846 -0.013 0.012 rpy=0 1.0471975512 0, axis 1.0 0.0 0.0
- added joint wheel60-roller4: type continuous, parent wheel-frame60, child roller-0-4, origin xyz=0.0 -0.013 -0.024 rpy=0 3.1415926536 0, axis 1.0 0.0 0.0
- added joint wheel60-roller5: type continuous, parent wheel-frame60, child roller-0-5, origin xyz=-0.0207846 -0.013 0.012 rpy=0 5.235987756 0, axis 1.0 0.0 0.0
